Commit message: Valkyrie working in CartesI/O

File: robots/valkyrie/urdf/valkyrie_sim_arm_mass_sims.urdf (robot description, URDF)
Before this commit: robot valkyrie, 50 links, 49 joints
Links:
- removed link head
- removed link head_hokuyo_frame
- removed link head_imu_link
- removed link left_led_frame
- removed link right_led_frame
- added link gaze, mass 1.41984; collision box size=0.0468 0.12 0.1184; collision box size=0.1311 0.12 0.0591
- added link gaze_hokuyo_frame, mass 1e-5
- added link gaze_imu_link, mass 1e-5; visual box size=0.01 0.01 0.01
- added link leftForearmLink, mass 2.476; collision mesh filename=package://tutorial_iros2018/robots/valkyrie/meshes/arms/aj5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; visual mesh filename=package://tutorial_iros2018/robots/valkyrie/meshes/arms/aj5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
- added link leftWristRollLink, mass 0.14; collision mesh filename=package://tutorial_iros2018/robots/valkyrie/meshes/arms/aj6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; visual mesh filename=package://tutorial_iros2018/robots/valkyrie/meshes/arms/aj6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
- added link rightForearmLink, mass 2.476; collision mesh filename=package://tutorial_iros2018/robots/valkyrie/meshes/arms/aj5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; visual mesh filename=package://tutorial_iros2018/robots/valkyrie/meshes/arms/aj5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
- added link rightWristRollLink, mass 0.14; collision mesh filename=package://tutorial_iros2018/robots/valkyrie/meshes/arms/aj6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; visual mesh filename=package://tutorial_iros2018/robots/valkyrie/meshes/arms/aj6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
- link pelvis: geometry collision mesh filename=package://tutorial_iros2018/robots/valkyrie/meshes/pelvis/p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; visual mesh filename=package://tutorial_iros2018/robots/valkyrie/meshes/pelvis/p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
Joints:
- removed joint head_hokuyo_joint
- removed joint head_imu_joint
- removed joint left_led_frame_joint
- removed joint multisense_head_root_joint
- removed joint right_led_frame_joint
- added joint gaze_hokuyo_joint: type fixed, parent hokuyo_link, child gaze_hokuyo_frame, origin xyz=0.03 0 0.015 rpy=0 0 0, axis 0 1 0
- added joint gaze_imu_joint: type fixed, parent gaze, child gaze_imu_link, origin xyz=-0.0475 0.035 0.0 rpy=0 0 0
- added joint leftForearmYaw: type revolute, parent leftElbowPitchLink, child leftForearmLink, origin xyz=-0.0254 0 0 rpy=0.0 0.0 0.0, axis 0 1 0, limit lower=-2.019 upper=3.14 effort=26 velocity=5
- added joint leftWristRoll: type revolute, parent leftForearmLink, child leftWristRollLink, origin xyz=0.0 0.2871 0.0 rpy=0.0 0.0 0.0, axis 1 0 0, limit lower=-0.62 upper=0.625 effort=14 velocity=1
- added joint multisense_gaze_root_joint: type fixed, parent upperNeckPitchLink, child gaze, origin xyz=0.183585961 0.0 0.075353826 rpy=-3.14159 0.130899694 0.0, axis 0 0 1
- added joint rightForearmYaw: type revolute, parent rightElbowPitchLink, child rightForearmLink, origin xyz=-0.0254 0 0 rpy=0.0 0.0 0.0, axis 0 1 0, limit lower=-2.019 upper=3.14 effort=26 velocity=5
- added joint rightWristRoll: type revolute, parent rightForearmLink, child rightWristRollLink, origin xyz=0.0 -0.2871 0.0 rpy=0.0 0.0 0.0, axis 1 0 0, limit lower=-0.625 upper=0.62 effort=14 velocity=1
- joint center_bottom_led_frame_joint: parent head -> gaze
- joint center_top_led_frame_joint: parent head -> gaze
- joint hokuyo_joint: axis 1 0 0 -> (none); parent head -> gaze; type continuous -> fixed
- joint left_camera_frame_joint: parent head -> gaze
- joint right_camera_frame_joint: parent head -> gaze
