Commit message: Working verion with CartesI/O

File: robots/reemc/reemc.urdf (robot description, URDF)
Before this commit: robot reemc, 55 links, 54 joints
Links:
- removed link hand_left_indication_link
- removed link hand_right_indication_link
- added link world
Joints:
- removed joint hand_left_indication_joint
- removed joint hand_right_indication_joint
- added joint reference: type floating, parent world, child base_link

Commit message: fix

File: robots/reemc/reemc.urdf (robot description, URDF)
Before this commit: robot reemc, 54 links, 53 joints
Links:
- added link l_leg_ft
- added link r_leg_ft
Joints:
- added joint l_leg_ft_joint: type fixed, parent leg_left_6_link, child l_leg_ft, origin xyz=0.0 0.0 0.0 rpy=0.0 0.0 0
- added joint r_leg_ft_joint: type fixed, parent leg_right_6_link, child r_leg_ft, origin xyz=0.0 0.0 0.0 rpy=0.0 0.0 0

Commit message: Added gaze task

File: robots/reemc/reemc.urdf (robot description, URDF)
Before this commit: robot reemc, 56 links, 55 joints
Links:
- removed link head_sonar_03_link
- added link gaze, mass 0.001
Joints:
- joint head_sonar_03_joint: child head_sonar_03_link -> gaze

Commit message: Added tutorial for qppvm control in opensot

File: robots/reemc/reemc.urdf (robot description, URDF)
Before this commit: robot reemc, 56 links, 55 joints
Links:
- added link Waist
Joints:
- added joint waist_joint: type fixed, parent base_link, child Waist
