Commit message: iCub Tutorial using XBotControl .

File: robots/iCub/iCub.urdf (robot description, URDF)
Before this commit: robot iCub, 56 links, 55 joints
Joints:
- joint l_ankle_pitch: limit lower=-0.733038 upper=0.366519 effort=24 velocity=100 -> lower=-0.733038 upper=0.366519 effort=24 velocity=3.14
- joint l_ankle_roll: limit lower=-0.418879 upper=0.418879 effort=11 velocity=100 -> lower=-0.418879 upper=0.418879 effort=11 velocity=3.14
- joint l_elbow: limit lower=0.0959931 upper=1.85005 effort=20 velocity=100 -> lower=0.0959931 upper=1.85005 effort=20 velocity=3.14
- joint l_hip_pitch: limit lower=-0.767945 upper=2.30383 effort=84 velocity=100 -> lower=-0.767945 upper=2.30383 effort=84 velocity=3.14
- joint l_hip_roll: limit lower=-2.07694 upper=0.296706 effort=84 velocity=100 -> lower=-2.07694 upper=0.296706 effort=84 velocity=3.14
- joint l_hip_yaw: limit lower=-1.37881 upper=1.37881 effort=40 velocity=100 -> lower=-1.37881 upper=1.37881 effort=40 velocity=3.14
- joint l_knee: limit lower=-2.18166 upper=0.401426 effort=30 velocity=100 -> lower=-2.18166 upper=0.401426 effort=30 velocity=3.14
- joint l_shoulder_pitch: limit lower=-1.65806 upper=0.0872665 effort=84 velocity=100 -> lower=-1.65806 upper=0.0872665 effort=84 velocity=3.14
- joint l_shoulder_roll: limit lower=0 upper=2.80649 effort=84 velocity=100 -> lower=0 upper=2.80649 effort=84 velocity=3.14
- joint l_shoulder_yaw: limit lower=-0.645772 upper=1.74533 effort=34 velocity=100 -> lower=-0.645772 upper=1.74533 effort=34 velocity=3.14
- joint l_wrist_pitch: limit lower=-1.13446 upper=0.174533 effort=0.65 velocity=100 -> lower=-1.13446 upper=0.174533 effort=0.65 velocity=3.14
- joint l_wrist_prosup: limit lower=-0.872665 upper=0.872665 effort=0.45 velocity=100 -> lower=-0.872665 upper=0.872665 effort=0.45 velocity=3.14
- joint l_wrist_yaw: limit lower=-0.436332 upper=0.436332 effort=0.65 velocity=100 -> lower=-0.436332 upper=0.436332 effort=0.65 velocity=3.14
- joint neck_pitch: limit lower=-0.698132 upper=0.523599 effort=20 velocity=100 -> lower=-0.698132 upper=0.523599 effort=20 velocity=3.14
- joint neck_roll: limit lower=-1.22173 upper=1.0472 effort=20 velocity=100 -> lower=-1.22173 upper=1.0472 effort=20 velocity=3.14
- joint neck_yaw: limit lower=-0.959931 upper=0.959931 effort=20 velocity=100 -> lower=-0.959931 upper=0.959931 effort=20 velocity=3.14
- joint r_ankle_pitch: limit lower=-0.733038 upper=0.366519 effort=24 velocity=100 -> lower=-0.733038 upper=0.366519 effort=24 velocity=3.14
- joint r_ankle_roll: limit lower=-0.418879 upper=0.418879 effort=11 velocity=100 -> lower=-0.418879 upper=0.418879 effort=11 velocity=3.14
- joint r_elbow: limit lower=0.0959931 upper=1.85005 effort=20 velocity=100 -> lower=0.0959931 upper=1.85005 effort=20 velocity=3.14
- joint r_hip_pitch: limit lower=-0.767945 upper=2.30383 effort=84 velocity=100 -> lower=-0.767945 upper=2.30383 effort=84 velocity=3.14
- joint r_hip_roll: limit lower=-2.07694 upper=0.296706 effort=84 velocity=100 -> lower=-2.07694 upper=0.296706 effort=84 velocity=3.14
- joint r_hip_yaw: limit lower=-1.37881 upper=1.37881 effort=40 velocity=100 -> lower=-1.37881 upper=1.37881 effort=40 velocity=3.14
- joint r_knee: limit lower=-2.18166 upper=0.401426 effort=30 velocity=100 -> lower=-2.18166 upper=0.401426 effort=30 velocity=3.14
- joint r_shoulder_pitch: limit lower=-1.65806 upper=0.0872665 effort=84 velocity=100 -> lower=-1.65806 upper=0.0872665 effort=84 velocity=3.14
- joint r_shoulder_roll: limit lower=0 upper=2.80649 effort=84 velocity=100 -> lower=0 upper=2.80649 effort=84 velocity=3.14
- joint r_shoulder_yaw: limit lower=-0.645772 upper=1.74533 effort=34 velocity=100 -> lower=-0.645772 upper=1.74533 effort=34 velocity=3.14
- joint r_wrist_pitch: limit lower=-1.13446 upper=0.174533 effort=0.65 velocity=100 -> lower=-1.13446 upper=0.174533 effort=0.65 velocity=3.14
- joint r_wrist_prosup: limit lower=-0.872665 upper=0.872665 effort=0.45 velocity=100 -> lower=-0.872665 upper=0.872665 effort=0.45 velocity=3.14
- joint r_wrist_yaw: limit lower=-0.436332 upper=0.436332 effort=0.65 velocity=100 -> lower=-0.436332 upper=0.436332 effort=0.65 velocity=3.14
- joint torso_pitch: limit lower=-0.383972 upper=1.46608 effort=36 velocity=100 -> lower=-0.383972 upper=1.46608 effort=36 velocity=3.14
- joint torso_roll: limit lower=-0.680678 upper=0.680678 effort=80 velocity=100 -> lower=-0.680678 upper=0.680678 effort=80 velocity=3.14
- joint torso_yaw: limit lower=-1.02974 upper=1.02974 effort=80 velocity=100 -> lower=-1.02974 upper=1.02974 effort=80 velocity=3.14
